Commit message: 简化了机器人碰撞模型

File: source/robot_lab/data/Robots/TQBot/TQBot2_description/urdf/TQBot2.urdf (robot description, URDF)
Before this commit: robot TQBot2, 31 links, 30 joints
Links:
- link FL_thigh: geometry collision cylinder length=0.213 radius=0.02; collision mesh filename=package://TQBot2_description/meshes/simple_thigh.STL scale=0.001 0.001 0.001
- link FR_thigh: geometry collision cylinder length=0.213 radius=0.02; collision mesh filename=package://TQBot2_description/meshes/simple_thigh.STL scale=0.001 0.001 0.001
- link RL_thigh: geometry collision cylinder length=0.213 radius=0.02; collision mesh filename=package://TQBot2_description/meshes/simple_thigh.STL scale=0.001 0.001 0.001
- link RR_thigh: geometry collision cylinder length=0.213 radius=0.02; collision mesh filename=package://TQBot2_description/meshes/simple_thigh.STL scale=0.001 0.001 0.001

Commit message: Refactor TQBot2 URDF and configuration files for improved locomotion - Removed the fixed base link from the URDF to enhance flexibility. - Updated joint limits for various joints to refine movement constraints. - Changed collider type in TQBot2 configuration from convex decomposition to convex hull. - Adjusted base link references in the rough environment configuration to align with the new URDF structure. - Modified terrain type settings for the rolling environment to improve simulation accuracy.

File: source/robot_lab/data/Robots/TQBot/TQBot2_description/urdf/TQBot2.urdf (robot description, URDF)
Before this commit: robot TQBot2, 31 links, 30 joints
Links:
- removed link base
Joints:
- removed joint floating_base
- joint FL_hip_joint: limit lower=-1.588 upper=1.588 effort=23.7 velocity=30.1 -> lower=-1.588 upper=0.3 effort=23.7 velocity=30.1
- joint FL_thigh_joint: limit lower=-3.141 upper=2.3 effort=23.7 velocity=30.1 -> lower=0.65 upper=2.3 effort=23.7 velocity=30.1
- joint FR_hip_joint: limit lower=-1.588 upper=1.588 effort=23.7 velocity=30.1 -> lower=-0.3 upper=1.588 effort=23.7 velocity=30.1
- joint FR_thigh_joint: limit lower=-3.141 upper=2.3 effort=23.7 velocity=30.1 -> lower=0.65 upper=2.3 effort=23.7 velocity=30.1
- joint RL_hip_joint: limit lower=-1.588 upper=1.588 effort=23.7 velocity=30.1 -> lower=-1.588 upper=0.3 effort=23.7 velocity=30.1
- joint RL_thigh_joint: limit lower=-3.141 upper=2.3 effort=23.7 velocity=30.1 -> lower=0.65 upper=2.3 effort=23.7 velocity=30.1
- joint RR_hip_joint: limit lower=-1.588 upper=1.588 effort=23.7 velocity=30.1 -> lower=-0.3 upper=1.588 effort=23.7 velocity=30.1
- joint RR_thigh_joint: limit lower=-3.141 upper=2.3 effort=23.7 velocity=30.1 -> lower=0.65 upper=2.3 effort=23.7 velocity=30.1
