Commit message: feat: add TQBot2 recovery training support

File: source/robot_lab/data/Robots/TQBot/TQBot2_description/urdf/TQBot2.urdf (robot description, URDF)
Before this commit: robot TQBot2, 30 links, 29 joints
Links:
- added link FL_knee_contact
- added link FR_knee_contact
- added link RL_knee_contact
- added link RR_knee_contact
- added link base; visual box size=0.001 0.001 0.001
- link FL_calf: geometry collision cylinder length=0.153 radius=0.008; collision sphere radius=0.020
- link FR_calf: geometry collision cylinder length=0.153 radius=0.008; collision sphere radius=0.020
- link RL_calf: geometry collision cylinder length=0.153 radius=0.008; collision sphere radius=0.020
- link RR_calf: geometry collision cylinder length=0.153 radius=0.008; collision sphere radius=0.020
- link trunk: geometry collision mesh filename=package://TQBot2_description/meshes/simple_Body.STL scale=1 0.95 1; visual mesh filename=package://TQBot2_description/meshes/base_link.STL.dae scale=1 1 1
Joints:
- added joint FL_knee_contact_joint: type fixed, parent FL_thigh, child FL_knee_contact, origin xyz=-0.02 0 -0.213 rpy=0 0 0
- added joint FR_knee_contact_joint: type fixed, parent FR_thigh, child FR_knee_contact, origin xyz=-0.02 0 -0.213 rpy=0 0 0
- added joint RL_knee_contact_joint: type fixed, parent RL_thigh, child RL_knee_contact, origin xyz=0.02 0 -0.213 rpy=0 0 0
- added joint RR_knee_contact_joint: type fixed, parent RR_thigh, child RR_knee_contact, origin xyz=0.02 0 -0.213 rpy=0 0 0
- added joint floating_base: type fixed, parent base, child trunk, origin xyz=0 0 0.0247 rpy=0 0 0
- joint FL_hip_joint: limit lower=-1.588 upper=0.3 effort=23.7 velocity=30.1 -> lower=-1.588 upper=1.588 effort=23.7 velocity=30.1
- joint FL_thigh_joint: limit lower=0.65 upper=2.3 effort=23.7 velocity=30.1 -> lower=-3.141 upper=6.108 effort=23.7 velocity=30.1
- joint FR_hip_joint: limit lower=-0.3 upper=1.588 effort=23.7 velocity=30.1 -> lower=-1.588 upper=1.588 effort=23.7 velocity=30.1
- joint FR_thigh_joint: limit lower=0.65 upper=2.3 effort=23.7 velocity=30.1 -> lower=-3.141 upper=6.108 effort=23.7 velocity=30.1
- joint RL_hip_joint: limit lower=-1.588 upper=0.3 effort=23.7 velocity=30.1 -> lower=-1.588 upper=1.588 effort=23.7 velocity=30.1
- joint RL_thigh_joint: limit lower=0.65 upper=2.3 effort=23.7 velocity=30.1 -> lower=-3.141 upper=6.108 effort=23.7 velocity=30.1
- joint RR_hip_joint: limit lower=-0.3 upper=1.588 effort=23.7 velocity=30.1 -> lower=-1.588 upper=1.588 effort=23.7 velocity=30.1
- joint RR_thigh_joint: limit lower=0.65 upper=2.3 effort=23.7 velocity=30.1 -> lower=-3.141 upper=6.108 effort=23.7 velocity=30.1
